Commit message: first commit

File: my_robot/urdf/my_robot.xacro (robot description, xacro)
@@ -26,5 +26,5 @@
    </link>
   <joint type="continuous"  name="left_wheel_hinge">
-    <origin xyz="0 0.12 0" rpy="0 0 0" />
+    <origin xyz="0 0.15 0" rpy="0 0 0" />
       <child link="left_wheel"/>
     <parent link="chassis"/>
@@ -57,5 +57,5 @@
   </link>
   <joint type="continuous" name="right_wheel_hinge">
-    <origin xyz="0 -0.12 0" rpy="0 0 0" />
+    <origin xyz="0 -0.15 0" rpy="0 0 0" />
       <child link="right_wheel"/>
   <parent link="chassis"/>
@@ -66,5 +66,5 @@
   <link name="robot_footprint"></link>
   <joint name="robot_footprint_joint" type="fixed">
-    <origin xyz="0 0 0" rpy="0 0 0" />
+    <origin xyz="0 0 0.1" rpy="0 0 0" />
     <parent link="robot_footprint"/>
     <child link="chassis" />
@@ -84,5 +84,5 @@
       <origin xyz="0 0 0" rpy=" 0 0 0"/>
       <geometry>
-        <box size=".6 .3 .1"/>
+        <box size=".6 .2 .1"/>
       </geometry>
     </collision>
@@ -90,5 +90,5 @@
       <origin xyz="0 0 0" rpy=" 0 0 0"/>
       <geometry>
-        <box size=".6 .3 .1"/>
+        <box size=".6 .2 .1"/>
       </geometry>
     </visual>
@@ -142,5 +142,5 @@
    </link>
   <joint type="fixed"  name="camera_joint">
-    <origin xyz="0.3 0 0" rpy="0 0 0" />
+    <origin xyz="0.2 0 0" rpy="0 0 0" />
       <child link="camera"/>
     <parent link="chassis"/>
